Commit message: Rename the 'mti-10' link to 'imu' to match IMU messages headers

File: urdf/warthog.urdf.xacro (robot description, xacro)
@@ -293,14 +293,14 @@
     <child link="imu_link" />
   </joint>
-  <link name="mti10" />
+  <link name="imu" />
   <joint name="mti10_joint" type="fixed">
     <origin xyz="0.43102 -0.1185 0.721" rpy="0 0 0" />
     <parent link="base_link" />
-    <child link="mti10" />
+    <child link="imu" />
   </joint>
   <link name="rslidar32" />
   <joint name="rslidar32_joint" type="fixed">
     <origin xyz="0.02632 0.1029 0.04536" rpy="0 0 0" />
-    <parent link="mti10" />
+    <parent link="imu" />
     <child link="rslidar32" />
   </joint>

Commit message: Update rslidar joint's parent to base_link

File: urdf/warthog.urdf.xacro (robot description, xacro)
@@ -301,6 +301,6 @@
   <link name="rslidar32" />
   <joint name="rslidar32_joint" type="fixed">
-    <origin xyz="0.02632 0.1029 0.04536" rpy="0 0 0" />
-    <parent link="imu" />
+    <origin xyz="0.45734 -0.0156 0.76636" rpy="0 0 0" />
+    <parent link="base_link" />
     <child link="rslidar32" />
   </joint>

Commit message: Add lidar - IMU pitch correction

File: urdf/warthog.urdf.xacro (robot description, xacro)
@@ -301,5 +301,5 @@
   <link name="rslidar32" />
   <joint name="rslidar32_joint" type="fixed">
-    <origin xyz="0.45734 -0.0156 0.76636" rpy="0 0 0" />
+    <origin xyz="0.45734 -0.0156 0.76636" rpy="0 028267838 0" /> <!-- pitch from 01/02/2023 FM calib data-->
     <parent link="base_link" />
     <child link="rslidar32" />

Commit message: Add missing decimal point

File: urdf/warthog.urdf.xacro (robot description, xacro)
@@ -301,5 +301,5 @@
   <link name="rslidar32" />
   <joint name="rslidar32_joint" type="fixed">
-    <origin xyz="0.45734 -0.0156 0.76636" rpy="0 028267838 0" /> <!-- pitch from 01/02/2023 FM calib data-->
+    <origin xyz="0.45734 -0.0156 0.76636" rpy="0 0.028267838 0" /> <!-- pitch from 01/02/2023 FM calib data-->
     <parent link="base_link" />
     <child link="rslidar32" />

Commit message: Move imu angle correction from lidar to imu joint

File: urdf/warthog.urdf.xacro (robot description, xacro)
@@ -295,5 +295,5 @@
   <link name="imu" />
   <joint name="mti10_joint" type="fixed">
-    <origin xyz="0.43102 -0.1185 0.721" rpy="0 0 0" />
+    <origin xyz="0.43102 -0.1185 0.721" rpy="0 0.028267838 0" />
     <parent link="base_link" />
     <child link="imu" />
@@ -301,5 +301,5 @@
   <link name="rslidar32" />
   <joint name="rslidar32_joint" type="fixed">
-    <origin xyz="0.45734 -0.0156 0.76636" rpy="0 0.028267838 0" /> <!-- pitch from 01/02/2023 FM calib data-->
+    <origin xyz="0.45734 -0.0156 0.76636" rpy="0 0 0" /> <!-- pitch from 01/02/2023 FM calib data-->
     <parent link="base_link" />
     <child link="rslidar32" />

Commit message: Added calibration description comment

File: urdf/warthog.urdf.xacro (robot description, xacro)
@@ -295,5 +295,5 @@
   <link name="imu" />
   <joint name="mti10_joint" type="fixed">
-    <origin xyz="0.43102 -0.1185 0.721" rpy="0 0.028267838 0" />
+    <origin xyz="0.43102 -0.1185 0.721" rpy="0 0.028267838 0" /> <!-- pitch from 01/02/2023 FM calib data-->
     <parent link="base_link" />
     <child link="imu" />
@@ -301,5 +301,5 @@
   <link name="rslidar32" />
   <joint name="rslidar32_joint" type="fixed">
-    <origin xyz="0.45734 -0.0156 0.76636" rpy="0 0 0" /> <!-- pitch from 01/02/2023 FM calib data-->
+    <origin xyz="0.45734 -0.0156 0.76636" rpy="0 0 0" />
     <parent link="base_link" />
     <child link="rslidar32" />

Commit message: Sync with humble version

File: urdf/warthog.urdf.xacro (robot description, xacro)
@@ -293,14 +293,14 @@
     <child link="imu_link" />
   </joint>
-  <link name="mti10" />
+  <link name="imu" />
   <joint name="mti10_joint" type="fixed">
-    <origin xyz="0.43102 -0.1185 0.721" rpy="0 0 0" />
-    <parent link="base_link" />
-    <child link="mti10" />
+    <origin xyz="0.43102 -0.1185 0.721" rpy="0 0.028267838 0" /> <!-- pitch from 01/02/2023 FM calib data-->
+    <parent link="base_link" />
+    <child link="imu" />
   </joint>
   <link name="rslidar32" />
   <joint name="rslidar32_joint" type="fixed">
-    <origin xyz="0.02632 0.1029 0.04536" rpy="0 0 0" />
-    <parent link="mti10" />
+    <origin xyz="0.45734 -0.0156 0.76636" rpy="0 0 0" />
+    <parent link="base_link" />
     <child link="rslidar32" />
   </joint>

Commit message: Sync imu frame name with mti10 imu message headers

File: urdf/warthog.urdf.xacro (robot description, xacro)
@@ -293,9 +293,9 @@
     <child link="imu_link" />
   </joint>
-  <link name="imu" />
+  <link name="mti10" />
   <joint name="mti10_joint" type="fixed">
     <origin xyz="0.43102 -0.1185 0.721" rpy="0 0.028267838 0" /> <!-- pitch from 01/02/2023 FM calib data-->
     <parent link="base_link" />
-    <child link="imu" />
+    <child link="mti10" />
   </joint>
   <link name="rslidar32" />

Commit message: Add previous calibration specification

File: urdf/warthog.urdf.xacro (robot description, xacro)
@@ -295,6 +295,6 @@
   <link name="mti10" />
   <joint name="mti10_joint" type="fixed">
-    <!-- <origin xyz="0.43102 -0.1185 0.721" rpy="0 0.028267838 0" /> -->
-    <origin xyz="0.43102 -0.1185 0.721" rpy="0 0.034338479 0" /> <!-- Calibration done on march 16th loop around vachon rosbag: rosbag2_2023_03_16-13_26_17 -->
+    <!-- <origin xyz="0.43102 -0.1185 0.721" rpy="0 0.028267838 0" /> --> <!-- Calibration on February 1th 2023 in FM-->
+    <origin xyz="0.43102 -0.1185 0.721" rpy="0 0.034338479 0" /> <!-- Calibration done on March 16th loop around vachon rosbag: rosbag2_2023_03_16-13_26_17 -->
     <parent link="base_link" />
     <child link="mti10" />

Commit message: Calibrated IMU-Lidar alignment

File: urdf/warthog.urdf.xacro (robot description, xacro)
@@ -295,5 +295,6 @@
   <link name="mti10" />
   <joint name="mti10_joint" type="fixed">
-    <origin xyz="0.43102 -0.1185 0.721" rpy="0 0.028267838 0" /> <!-- pitch from 01/02/2023 FM calib data-->
+    <!-- <origin xyz="0.43102 -0.1185 0.721" rpy="0 0.028267838 0" /> -->
+    <origin xyz="0.43102 -0.1185 0.721" rpy="0 0.034338479 0" /> <!-- Calibration done on march 16th loop around vachon rosbag: rosbag2_2023_03_16-13_26_17 -->
     <parent link="base_link" />
     <child link="mti10" />

Commit message: WD Modified imu pitch value from calib done on humble

File: urdf/warthog.urdf.xacro (robot description, xacro)
@@ -295,5 +295,5 @@
   <link name="mti10" />
   <joint name="mti10_joint" type="fixed">
-    <origin xyz="0.43102 -0.1185 0.721" rpy="0 0.028267838 0" /> <!-- pitch from 01/02/2023 FM calib data-->
+    <origin xyz="0.43102 -0.1185 0.721" rpy="0 0.034338479 0" /> <!-- pitch from 01/02/2023 FM calib data-->
     <parent link="base_link" />
     <child link="mti10" />

Commit message: Add footprint_link

File: urdf/warthog.urdf.xacro (robot description, xacro)
@@ -224,4 +224,10 @@
     <child link="chassis_link" />
   </joint>
+  <link name="footprint_link"></link>
+  <joint name="footprint_joint" type="fixed">
+    <origin xyz="0 0 -${wheel_radius}" rpy="0 0 0" />
+    <parent link="base_link"/>
+    <child link="footprint_link" />
+  </joint>
   <link name="chassis_link">
     <inertial>

Commit message: added link for radar with no transform values(0 everywhere)

File: urdf/warthog.urdf.xacro (robot description, xacro)
@@ -312,4 +312,10 @@
     <child link="rslidar32" />
   </joint>
+  <link name="radar" />
+  <joint name="radar_joint" type="fixed">
+    <origin xyz="0 0 0" rpy="0 0 0" />
+    <parent link="base_link" />
+    <child link="radar" />
+  </joint>
   <link name="rslidar16_left" />
   <joint name="rslidar16_left_joint" type="fixed">

Commit message: added dummy camera link

File: urdf/warthog.urdf.xacro (robot description, xacro)
@@ -318,4 +318,10 @@
     <child link="radar" />
   </joint>
+  <link name="basler_camera" />
+  <joint name="basler_camera_joint" type="fixed">
+    <origin xyz="0 0 0" rpy="0 0 0" />
+    <parent link="base_link" />
+    <child link="basler_camera" />
+  </joint>
   <link name="rslidar16_left" />
   <joint name="rslidar16_left_joint" type="fixed">

Commit message: Added both dps310 frames.

File: urdf/warthog.urdf.xacro (robot description, xacro)
@@ -312,4 +312,16 @@
     <child link="rslidar32" />
   </joint>
+  <link name="dps310_1" />
+  <joint name="dps310_1_joint" type="fixed">
+    <origin xyz="-0.561975 0.301228 -0.25686" rpy="0 0 0" />
+    <parent link="rslidar32" />
+    <child link="dps310_1" />
+  </joint>
+  <link name="dps310_2" />
+  <joint name="dps310_2_joint" type="fixed">
+    <origin xyz="-0.244475 0.301228 -0.19986" rpy="0 0 0" />
+    <parent link="rslidar32" />
+    <child link="dps310_2" />
+  </joint>
   <link name="radar" />
   <joint name="radar_joint" type="fixed">

Commit message: update urdf

File: urdf/warthog.urdf.xacro (robot description, xacro)
@@ -301,6 +301,6 @@
   <link name="mti10" />
   <joint name="mti10_joint" type="fixed">
-    <!-- <origin xyz="0.43102 -0.1185 0.721" rpy="0 0.028267838 0" /> --> <!-- Calibration on February 1th 2023 in FM-->
-    <origin xyz="0.43102 -0.1185 0.721" rpy="0 0.034338479 0" /> <!-- Calibration done on March 16th loop around vachon rosbag: rosbag2_2023_03_16-13_26_17 -->
+    <!--  <origin xyz="0.43102 -0.1185 0.721" rpy="0 0.034338479 0" /> Calibration done on March 16th loop around vachon rosbag: rosbag2_2023_03_16-13_26_17 -->
+    <origin xyz="0.43102 -0.1185 0.721" rpy="0 0.001 0" /> <!-- Calibration done on the warthog_first_experiment_mobile_lab_to_main_building_clipped rosbag -->
     <parent link="base_link" />
     <child link="mti10" />

Commit message: Update imu-lidar angle

File: urdf/warthog.urdf.xacro (robot description, xacro)
@@ -301,6 +301,5 @@
   <link name="mti10" />
   <joint name="mti10_joint" type="fixed">
-    <!--  <origin xyz="0.43102 -0.1185 0.721" rpy="0 0.034338479 0" /> Calibration done on March 16th loop around vachon rosbag: rosbag2_2023_03_16-13_26_17 -->
-    <origin xyz="0.43102 -0.1185 0.721" rpy="0 0.001 0" /> <!-- Calibration done on the warthog_first_experiment_mobile_lab_to_main_building_clipped rosbag -->
+    <origin xyz="0.43102 -0.1185 0.721" rpy="0 0 0" />
     <parent link="base_link" />
     <child link="mti10" />
